File: pcb/BansheeNornV5.sch (EAGLE design)
At the start: 93 parts, among them IC1 ESP32-S3-WROOM-1-N8, IC2 MAX8647ETE+, IC3 LSM6DS3USTR, IC5 NCV8163ASN330T1G, IC6 DG2034EDN-T1-GE4, IC7 BCR421UFD-7, IC8 DRV8835DSSR, Q1 LTR-4206E, Q10 IRFML8244TRPBF, Q2 SI3493DDV-T1-GE3, Q3 IRFML8244TRPBF, Q4 LTR-4206E, Q5 LTR-4206E, Q6 LTR-4206E, Q7 LTR-4206E, Q8 LTR-4206E, Y1 XRCGB40M000F5A00R0

Commit message: update: readme
Parts:
- removed C10: 22uF, Capacitor:C3216
- removed C15: 0.1u, Capacitor:C1005
- removed IC5: NCV8163ASN330T1G, NCV8163ASN330T1G:NCV8163ASN330T1G
- removed IC8: DRV8835DSSR, DRV8835DSSR:DRV8835DSSR
- removed Q10: IRFML8244TRPBF, IRFML8244TRPBF:IRFML8244TRPBF
- removed Q6: LTR-4206E, LTR-4206E:LTR-4206E
- added C18: 0.1u, Capacitor:C1005
- added IC4: NCV8163ASN330T1G, NCV8163ASN330T1G:NCV8163ASN330T1G
- added R26, R27, R28, R29, R30, R31, R32, R33, R6: 18, Resistor:R1608
- added U$32: PAD, pad:PAD
- added U1: LXDC55FAAA-203, LXDC55FAAA-203:LXDC55FAAA-203
- C13: value (none) -> 0.1u; device Capacitor:C3216 -> Capacitor:C1005
- C14: value 22uF -> (none)
- C4, C6: value 12pF -> (none); device Capacitor:C1005 -> Capacitor:C3216
- C8: value 10uF -> 0.1u; device Capacitor:C3216 -> Capacitor:C1005
- C9: value 100pF -> (none); device Capacitor:C1005 -> Capacitor:C1608
- Q5: value LTR-4206E -> SI3460DDV-T1-GE3; device LTR-4206E:LTR-4206E -> SI3460DDV-T1-GE3:SI3460DDV-T1-GE3
- R10: value 10k -> 18; device Resistor:R1005 -> Resistor:R1608
- R12, R13, R4: value 100k -> 10k
- R15: value 1k -> 18; device Resistor:R1005 -> Resistor:R1608
- R21: value 1k -> 10k
- R25: value 13~20k -> 18; device Resistor:R1005 -> Resistor:R1608
- R5: value 50 -> 0.5k
- U$1, U$11, U$17, U$20, U$8, U$9: value SENSOR_FRONT_PAD2 -> PAD; device sensor_front_pad2:SENSOR_FRONT_PAD2 -> pad:PAD
- U$10: value ENCORDER_1 -> SFH4550; device endorder_R:ENCORDER_1 -> LED:SFH4550
- U$12, U$24: value ENCORDER_1 -> PANA; device endorder_R:ENCORDER_1 -> con_tantal_pana:PANA
- U$16: value SFH4550 -> PANA; device LED:SFH4550 -> con_tantal_pana:PANA
- U$18: value PAD -> TB6614; device pad:PAD -> SSOP16:TB6614
- U$22: value ENCORDER_1 -> TB6614; device endorder_R:ENCORDER_1 -> SSOP16:TB6614
- U$3: value MUN12AD01-SG -> PANA; device MUN12AD01-SG:MUN12AD01-SG -> con_tantal_pana:PANA
- U$5, U$7: value SENSOR_FRONT_PAD2 -> PANA; device sensor_front_pad2:SENSOR_FRONT_PAD2 -> con_tantal_pana:PANA
Connections:
- removed net N$27: Q8.E, U$10.P$5
- removed net N$28: C9.2, R25.2, U$3.FB
- removed net N$30: IC8.AOUT1, U$29.P$1
- removed net N$31: Q7.E, U$11.P$1
- removed net N$34: Q7.C, U$11.P$2
- removed net N$38: U$10.P$3, U$16.A
- removed net N$61: IC8.BOUT2, U$57.P$1
- removed net SEN_L45: IC1.GPIO17, R17.2, U$22.P$1
- removed net SEN_R45_2: IC1.XTAL_32K_N, R15.2, U$24.P$5
- new net A_CW_CCW2: IC1.MTDO, U$18.IN2
- new net B_CW_CCW1: IC1.MTDI, U$22.IN2
- new net N$11: R28.1, U$25.P$1
- new net N$22: IC1.GPIO21, R4.1
- new net N$23: U$11.P$1, U$27.P$1, U$3.P$2
- net +3V3: now also C13.2, C14.2, C18.2, C4.2, C8.1, IC4.OUT, IC6.EN, IC6.V+, Q1.C, Q4.C, Q7.C, Q8.C, R15.1, R25.1, R26.1, R27.2, R28.2, R29.1, R30.2, R31.2, R32.2, R33.2, R8.2, U$18.STBY, U$18.VCC, U$22.STBY, U$22.VCC, U$24.P$2; no longer C1.2, C15.1, IC5.OUT, IC8.MODE, IC8.VCC, R5.2, R8.1, U$19.P$1, U$21.P$1, U$22.P$3, U$23.P$1, U$24.P$4, U$25.P$1, U$30.P$1, U$31.P$1, U$5.P$1, U$7.P$2
- net +5V: now also C1.2, C6.2, IC4.EN, IC4.IN, R10.1, U1.VOUT_1, U1.VOUT_2, U1.VOUT_3; no longer C10.2, C9.1, IC5.EN, IC5.IN, IC6.EN, IC6.V+, U$20.P$2, U$22.P$4, U$24.P$3, U$3.VOUT, U$8.P$1
- net A_CW_CCW: now also IC1.MTCK, U$18.IN1; no longer IC1.MTDI, IC8.AIN1_/_APHASE
- net A_PWM: now also IC1.GPIO38, U$18.PWM; no longer IC1.MTMS, IC8.AIN2_/_AENBL
- net B_CW_CCW: now also IC1.MTMS, U$22.IN1; no longer IC1.GPIO45, IC8.BIN1_/_BPHASE
- net B_PWM: now also U$22.PWM; no longer IC8.BIN2_/_BENBL
- net ENC_L_A: now also IC1.GPIO8; no longer IC1.GPIO12
- net ENC_L_B: now also IC1.GPIO9; no longer IC1.GPIO13
- net ENC_L_CLK: now also IC1.GPIO7; no longer IC1.GPIO11
- net ENC_L_CS: now also IC1.GPIO37; no longer IC1.GPIO10
- net GND: now also C14.1, C18.1, C4.1, C6.1, C9.1, IC4.GND, Q5.S, R21.2, R5.2, R6.1, U$12.P$1, U$16.P$1, U$18.GND, U$18.PGND1, U$18.PGND2, U$22.GND, U$22.PGND1, U$22.PGND2, U$24.P$1, U$5.P$1, U1.GND_1, U1.GND_2, U1.GND_3, U1.GND_4; no longer C10.1, C14.2, C15.2, C4.2, C6.2, IC5.GND, IC8.GND_1, IC8.GND_2, Q10.S, R10.2, R15.1, R21.1, R25.1, U$2.P$2, U$3.GND
- net L45_CATHODE: now also U$14.K; no longer U$22.P$5
- net L90_CATHODE: now also U$44.K; no longer U$8.P$2
- net LED_A0: now also IC1.GPIO11; no longer IC1.GPIO8
- net LED_A1: now also IC1.GPIO12; no longer IC1.GPIO9
- net LED_EN: now also IC1.GPIO10; no longer IC1.GPIO7
- net LED_SCL: now also IC1.GPIO14; no longer IC1.GPIO37
- net LED_SDA: now also IC1.XTAL_32K_N; no longer IC1.GPIO36
- net N$1: now also R10.2; no longer R5.1
- net N$10: now also R30.1, U$19.P$1; no longer U$44.K, U$9.P$1
- net N$12: now also IC1.GPIO19, R4.2; no longer IC8.AOUT2, U$26.P$1
- net N$13: now also U$17.P$1, U$22.O2_1, U$22.O2_2, U$7.P$1; no longer IC8.BOUT1, U$27.P$1
- net N$14: now also R27.1, U$31.P$1; no longer Q5.E, U$12.P$6
- net N$16: now also C9.2, IC4.NC; no longer Q4.E, U$12.P$5
- net N$18: now also R29.2, U$14.A; no longer Q4.C, Q5.C, U$12.P$4
- net N$19: now also R15.2, U$10.A; no longer D2.A, Q10.D, U$58.P$1
- net N$20: now also R25.2, U$44.A; no longer U$10.P$2, U$16.K
- net N$21: now also R26.2, U$4.A; no longer U$12.P$3, U$14.A
- net N$24: now also U$26.P$1, U$57.P$1, U$7.P$2; no longer Q6.E, U$10.P$6
- net N$26: now also R5.1, U1.FB; no longer U$17.P$1, U$4.A
- net N$29: now also D2.A, Q5.D_1, Q5.D_2, Q5.D_3, Q5.D_4, U$58.P$1; no longer U$17.P$2, U$4.K
- net N$32: no longer C4.1
- net N$33: no longer C6.1
- net N$36: now also U$1.P$1, U$18.O2_1, U$18.O2_2, U$32.P$1; no longer Q6.C, Q8.C, U$10.P$4
- net N$37: now also U$22.O1_1, U$22.O1_2, U$29.P$1, U$8.P$1; no longer U$12.P$2, U$14.K
- net N$4: now also R6.2, U$2.P$2; no longer R4.2, U$2.P$1
- net N$6: now also U$18.O1_1, U$18.O1_2, U$3.P$1, U$9.P$1; no longer IC1.MTCK
- net N$7: now also R33.1, U$30.P$1; no longer Q1.C, U$1.P$1
- net N$8: now also R32.1, U$23.P$1; no longer Q1.E, U$1.P$2
- net N$9: now also R31.1, U$21.P$1; no longer U$44.A, U$9.P$2
- net R45_CATHODE: now also U$10.K; no longer U$24.P$2
- net R90_CATHODE: now also U$4.K; no longer U$20.P$1
- net SEN_L45_2: now also Q4.E, R17.2; no longer R21.2, U$22.P$2
- net SEN_L90: now also IC1.XTAL_32K_P, Q1.E; no longer IC1.GPIO19, U$7.P$1
- net SEN_R45: now also IC1.GPIO17, Q8.E; no longer IC1.XTAL_32K_P, U$24.P$6
- net SEN_R90: now also IC1.GPIO13, Q7.E; no longer IC1.GPIO14, U$5.P$2
- net SUCTION_PWM: now also IC1.GPIO35, Q5.G, R21.1; no longer IC1.MTDO, Q10.G, R10.1
- net SW1: now also IC1.GPIO34, R8.1; no longer IC1.GPIO38, R8.2
- net VCC: now also U$12.P$2, U$16.P$2, U$18.VM_1, U$18.VM_2, U$2.P$1, U$20.P$1, U$22.VM_1, U$22.VM_2, U$5.P$2, U1.EN, U1.VIN_1, U1.VIN_2, U1.VIN_3; no longer C13.2, C14.1, C8.1, IC8.VM, R4.1, U$18.P$1, U$3.EN, U$3.VIN
Other:
- moved on the sheet: C13, C14, C4, C6, C8, CN2, Q1, Q4, Q7, U$14, U$4, U$44
